Commit message: added components to allow gazebo simulation

File: catkin_ws/src/pongbot/urdf/pongbot.urdf (robot description, URDF)
Before this commit: robot pongbot, 19 links, 18 joints
Links:
- added link dummy_root; visual box size=.2032 .2032 .0127
- link base_1: mass None -> 0.047
- link base_2: mass None -> 0.041
- link base_3_rim: mass None -> 0.016
- link base_3_turntable: mass None -> 0.017
- link bfemale_link1: mass None -> 0.011
- link elbow_motor: mass None -> 0.0535
- link elbow_rot: mass None -> 0
- link ffemale_link1: mass None -> 0.010
- link left_link2: mass None -> 0.007
- link lmale_link1: mass None -> 0.007
- link paddle: mass None -> 0.037
- link paddle_holder: mass None -> 0.021
- link paddle_motor: mass None -> 0.0535
- link paddle_rot: mass None -> 0
- link pan_motor: mass None -> 0.0535
- link right_link2: mass None -> 0.007
- link rmale_link1: mass None -> 0.007
- link steel_plate: mass None -> 4.211; geometry collision box size=.2032 .2032 .0127; visual box size=.2032 .2032 .0127
- link tilt_motor: mass None -> 0.0535
Joints:
- added joint dummy_to_steel: type fixed, parent dummy_root, child steel_plate, origin xyz=0 0 0
- joint elbow_joint: limit lower=0 upper=-3.14159 effort=1000.0 velocity=0.5 -> lower=-2.96705 upper=0 effort=1.5 velocity=0.5
- joint paddle_joint: limit (none) -> effort=1.5 velocity=1.0
- joint pan_joint: limit lower=-2.61799 upper=2.61799 effort=1000.0 velocity=0.5 -> lower=-2.61799 upper=2.61799 effort=1.5 velocity=0.5
- joint tilt_joint: limit lower=0 upper=3.14159 effort=1000.0 velocity=0.5 -> lower=0 upper=3.14159 effort=1.5 velocity=0.5
